Commit message: Added RViz2 and sanity check for filter performance

File: src/geodesic_description/urdf/simple_quadcopter.urdf.xacro (robot description, xacro)
@@ -54,5 +54,5 @@
         <parent link="base_link"/>
         <child link="imu"/>
-        <origin xyz="0 0 0" rpy="0 0 0"/>
+        <origin xyz="0 0 0" rpy="${pi} 0 0"/>
     </joint>
     <!-- Arm Macro -->
